Commit message: urdf file changes for gps and kinect sensor

File: turtlebot3_description/urdf/turtlebot3_waffle_pi.gazebo.xacro (robot description, xacro)
@@ -6,4 +6,22 @@
   <gazebo reference="base_link">
     <material>Gazebo/DarkGrey</material>
+  </gazebo>
+ <!-- Adding the kinect sensor -->
+<xacro:include filename="$(find kinect_v2)/urdf/kinect_v2.urdf.xacro" />
+  <xacro:kinect_v2  parent="base_link">
+    <origin xyz="-0.05 0 0.1" rpy="0 0 0"/>
+ </xacro:kinect_v2>
+ <gazebo>
+    <plugin name="gps_controller" filename="libhector_gazebo_ros_gps.so">
+      <alwayson>true</alwayson>
+      <updaterate>1.0</updaterate>
+      <bodyname>base_link</bodyname>
+      <topicname>/fix</topicname>
+      <velocitytopicname>/fix_velocity</velocitytopicname>
+      <drift>5.0 5.0 5.0</drift>
+      <gaussiannoise>0.1 0.1 0.1</gaussiannoise>
+      <velocitydrift>0 0 0</velocitydrift>
+      <velocitygaussiannoise>0.1 0.1 0.1</velocitygaussiannoise>
+    </plugin>
   </gazebo>
   <gazebo reference="wheel_left_link">
